Commit message: applied new changes to ur
Signed-off-by: Jakub Delicat <jakub.delicat@husarion.com>

File: urdf/ur.urdf.xacro (robot description, xacro)
@@ -18,5 +18,5 @@
   <xacro:macro name="ur"
     params="parent_link xyz rpy
-          tf_prefix:=None
+          device_namespace:=None
           ur_type:=ur3e">
     <xacro:include
@@ -24,4 +24,10 @@
       ns="ur_manipulator"
     />
+    <xacro:if value="${device_namespace == 'None'}">
+      <xacro:property name="prefix" value="" />
+    </xacro:if>
+    <xacro:unless value="${device_namespace == 'None'}">
+      <xacro:property name="prefix" value="${device_namespace}_" />
+    </xacro:unless>
     <xacro:property name="joint_limit_params"
       value="$(find ur_description)/config/${ur_type}/joint_limits.yaml" scope="parent" />
@@ -39,5 +45,5 @@
     <xacro:ur_manipulator.ur_robot
       name="${ur_type}"
-      tf_prefix="${tf_prefix}"
+      tf_prefix="${prefix}"
       parent="${parent_link}"
       joint_limits_parameters_file="${joint_limit_params}"
@@ -50,9 +56,9 @@
       <origin xyz="${xyz}" rpy="${rpy}" />
     </xacro:ur_manipulator.ur_robot>
-    <ros2_control name="${tf_prefix + ur_type}" type="system">
+    <ros2_control name="${prefix + ur_type}" type="system">
       <hardware>
         <plugin>ign_ros2_control/IgnitionSystem</plugin>
       </hardware>
-      <joint name="${tf_prefix}shoulder_pan_joint">
+      <joint name="${prefix}shoulder_pan_joint">
         <command_interface name="position">
           <param name="min">{-2*pi}</param>
@@ -70,5 +76,5 @@
         <state_interface name="effort" />
       </joint>
-      <joint name="${tf_prefix}shoulder_lift_joint">
+      <joint name="${prefix}shoulder_lift_joint">
         <command_interface name="position">
           <param name="min">{-2*pi}</param>
@@ -86,5 +92,5 @@
         <state_interface name="effort" />
       </joint>
-      <joint name="${tf_prefix}elbow_joint">
+      <joint name="${prefix}elbow_joint">
         <command_interface name="position">
           <param name="min">{-pi}</param>
@@ -102,5 +108,5 @@
         <state_interface name="effort" />
       </joint>
-      <joint name="${tf_prefix}wrist_1_joint">
+      <joint name="${prefix}wrist_1_joint">
         <command_interface name="position">
           <param name="min">{-2*pi}</param>
@@ -118,5 +124,5 @@
         <state_interface name="effort" />
       </joint>
-      <joint name="${tf_prefix}wrist_2_joint">
+      <joint name="${prefix}wrist_2_joint">
         <command_interface name="position">
           <param name="min">{-2*pi}</param>
@@ -134,5 +140,5 @@
         <state_interface name="effort" />
       </joint>
-      <joint name="${tf_prefix}wrist_3_joint">
+      <joint name="${prefix}wrist_3_joint">
         <command_interface name="position">
           <param name="min">{-2*pi}</param>
