Commit message: fixed astra
Signed-off-by: Jakub Delicat <jakub.delicat@husarion.com>

File: urdf/orbbec_astra.urdf.xacro (robot description, xacro)
@@ -19,4 +19,10 @@
       <xacro:property name="prefix" value="${tf_prefix}_" />
     </xacro:unless>
+    <joint name="${parent_link.rstrip('_link')}_to_${prefix}${camera_name}_joint" type="fixed">
+      <origin xyz="${xyz}" rpy="${rpy}" />
+      <parent link="${parent_link}" />
+      <child link="${prefix}${camera_name}_link" />
+    </joint>
+    <link name="${prefix}${camera_name}_link" />
     <joint name="${parent_link.rstrip('_link')}_to_${prefix}${camera_name}_orbbec_astra_joint" type="fixed">
       <origin xyz="${xyz}" rpy="${rpy}" />
@@ -55,5 +61,5 @@
     <joint name="${parent_link.rstrip('_link')}_to_${prefix}${camera_name}_color_joint" type="fixed">
       <origin xyz="-0.002 0.0125 0.03325" rpy="-0.003 0.0 -0.003" />
-      <parent link="${parent_link}" />
+      <parent link="${prefix}${camera_name}_link" />
       <child link="${prefix}${camera_name}_color_frame" />
     </joint>
@@ -61,5 +67,5 @@
     <joint name="${parent_link.rstrip('_link')}_to_${prefix}${camera_name}_depth_joint" type="fixed">
       <origin xyz="0.0 0.0 0.03325" rpy="0.0 0.0 0.0" />
-      <parent link="${parent_link}" />
+      <parent link="${prefix}${camera_name}_link" />
       <child link="${prefix}${camera_name}_depth_frame" />
     </joint>

Commit message: fixed astra
Signed-off-by: Jakub Delicat <jakub.delicat@husarion.com>

File: urdf/orbbec_astra.urdf.xacro (robot description, xacro)
@@ -22,5 +22,5 @@
       <child link="${device_namespace}_orbbec_astra_link" />
     </joint>
-    <link name="${device_namespace}_orbbec_astra">
+    <link name="${device_namespace}_orbbec_astra_link">
       <visual>
         <origin xyz="0.0 0.0 0.0" rpy="0.0 0.0 0.0" />
@@ -75,5 +75,5 @@
     </joint>
     <link name="${device_namespace}_color_optical_frame" />
-    <gazebo reference="${device_namespace}_orbbec_astra_link">
+    <gazebo reference="${device_namespace}_link">
       <!-- https://github.com/orbbec/OrbbecSDK_ROS2#all-available-topics -->
       <sensor type="camera" name="${ns}${device_namespace}_orbbec_astra_color">
