Commit message: revert cam link distance
Signed-off-by: Jakub Delicat <jakub.delicat@husarion.com>

File: urdf/stereolabs_zed.urdf.xacro (robot description, xacro)
@@ -110,5 +110,5 @@
       <parent link="${device_namespace}_center" />
       <child link="${device_namespace}_center_optical_frame" />
-      <origin xyz="0.05 0 0" rpy="0 0 0" />
+      <origin xyz="0.01 0 0" rpy="0 0 0" />
     </joint>
     <!-- Left Camera -->
