Commit message: renamed files
Signed-off-by: Jakub Delicat <jakub.delicat@husarion.com>

File: urdf/components.urdf.xacro (robot description, xacro)
@@ -82,4 +82,34 @@
         />
       </xacro:if>
+      <xacro:if value="${type == 'LDR13'}">
+        <xacro:include
+          filename="$(find ros_components_description)/urdf/ouster_os1_32.urdf.xacro"
+          ns="lidar"
+        />
+        <xacro:lidar.ouster_os1_32
+          parent_link="${parent_link}"
+          xyz="${xyz}"
+          rpy="${rpy}"
+          tf_prefix="${tf_prefix}"
+          use_gpu="${use_gpu}"
+          simulation_engine="${simulation_engine}"
+          namespace="${fixed_namespace}"
+        />
+      </xacro:if>
+      <xacro:if value="${type == 'LDR20'}">
+        <xacro:include
+          filename="$(find ros_components_description)/urdf/velodyne_puck.urdf.xacro"
+          ns="lidar"
+        />
+        <xacro:lidar.velodyne_puck
+          parent_link="${parent_link}"
+          xyz="${xyz}"
+          rpy="${rpy}"
+          tf_prefix="${tf_prefix}"
+          use_gpu="${use_gpu}"
+          simulation_engine="${simulation_engine}"
+          namespace="${fixed_namespace}"
+        />
+      </xacro:if>
       <xacro:if value="${index}">
         <xacro:load_componenet

File: urdf/ouster_os1_32.urdf.xacro (robot description, xacro)
@@ -5,7 +5,14 @@
                        use_gpu:=false
                        tf_prefix:=None
-                       topic:=os_lidar
+                       namespace:=None
+                       topic:=ouster/points
                        frame_id:=os_lidar
                        simulation_engine:=gazebo-classic">
+    <xacro:if value="${namespace == 'None'}">
+      <xacro:property name="ns" value="" />
+    </xacro:if>
+    <xacro:unless value="${namespace == 'None'}">
+      <xacro:property name="ns" value="${namespace}/" />
+    </xacro:unless>
     <xacro:if value="${use_gpu}">
       <xacro:property name="ray_type" value="gpu_ray" />
@@ -55,5 +62,5 @@
     <link name="${prefix}${frame_id}" />
     <gazebo reference="${prefix}${frame_id}">
-      <sensor type="${ray_type}" name="${prefix}ouster_os1_32_sensor">
+      <sensor type="${ray_type}" name="${ns}${prefix}ouster_os1_32_sensor">
         <visualize>false</visualize>
         <ray>
@@ -84,12 +91,20 @@
         </ray>
         <update_rate>20.0</update_rate>
-        <plugin name="${prefix}ouster_os1_32_${ray_type}" filename="libgazebo_ros_ray_sensor.so">
-          <ros>
-            <namespace></namespace>
-            <remapping>~/out:=${topic}</remapping>
-          </ros>
-          <output_type>sensor_msgs/PointCloud2</output_type>
-          <frame_name>${prefix}${frame_id}</frame_name>
-        </plugin>
+        <xacro:if value="${simulation_engine == 'ignition-gazebo'}">
+          <topic>${ns}${topic}</topic>
+          <frame_id>${prefix}${frame_id}</frame_id>
+          <ignition_frame_id>${prefix}${frame_id}</ignition_frame_id>
+          <always_on>true</always_on>
+        </xacro:if>
+        <xacro:if value="${simulation_engine == 'gazebo-classic'}">
+          <plugin name="${prefix}ouster_os1_32_${ray_type}" filename="libgazebo_ros_ray_sensor.so">
+            <ros>
+              <namespace>${ns}</namespace>
+              <remapping>~/out:=${topic}</remapping>
+            </ros>
+            <output_type>sensor_msgs/PointCloud2</output_type>
+            <frame_name>${prefix}${frame_id}</frame_name>
+          </plugin>
+        </xacro:if>
       </sensor>
     </gazebo>

File: urdf/velodyne_puck.urdf.xacro (robot description, xacro)
@@ -5,7 +5,7 @@
                        use_gpu:=false
                        tf_prefix:=None
-                       topic:=scan
+                       namespace:=None
+                       topic:=velodyne_points
                        frame_id:=velodyne
-                       namespace:=None
                        simulation_engine:=gazebo-classic">
     <xacro:if value="${namespace == 'None'}">

Commit message: Added ur
Signed-off-by: Jakub Delicat <jakub.delicat@husarion.com>

File: urdf/components.urdf.xacro (robot description, xacro)
@@ -29,5 +29,6 @@
       </xacro:if>
       <xacro:unless value="${device_namespace == 'None' and robot_namespace == 'None'}">
-        <xacro:property name="fixed_namespace" value="/${robot_namespace + device_namespace}" scope="parent" />
+        <xacro:property name="fixed_namespace" value="/${robot_namespace + device_namespace}"
+          scope="parent" />
       </xacro:unless>
       <xacro:if value="${device_namespace == 'None' and robot_namespace != 'None'}">
@@ -112,4 +113,30 @@
         />
       </xacro:if>
+      <xacro:if value="${type == 'MAN01'}">
+        <xacro:include
+          filename="$(find ros_components_description)/urdf/ur.urdf.xacro"
+          ns="manipulator"
+        />
+        <xacro:manipulator.ur
+          parent_link="${parent_link}"
+          xyz="${xyz}"
+          rpy="${rpy}"
+          tf_prefix="${tf_prefix}"
+          ur_type="ur3e"
+        />
+      </xacro:if>
+      <xacro:if value="${type == 'MAN02'}">
+        <xacro:include
+          filename="$(find ros_components_description)/urdf/ur.urdf.xacro"
+          ns="manipulator"
+        />
+        <xacro:manipulator.ur
+          parent_link="${parent_link}"
+          xyz="${xyz}"
+          rpy="${rpy}"
+          tf_prefix="${tf_prefix}"
+          ur_type="ur5e"
+        />
+      </xacro:if>
       <xacro:if value="${index}">
         <xacro:load_componenet

Commit message: Added rootiq
Signed-off-by: Jakub Delicat <jakub.delicat@husarion.com>

File: urdf/components.urdf.xacro (robot description, xacro)
@@ -204,4 +204,28 @@
         />
       </xacro:if>
+      <xacro:if value="${type == 'GRP02'}">
+        <xacro:include filename="$(find robotiq_description)/urdf/robotiq_2f_85_macro.urdf.xacro"
+          ns="gripper" />
+        <xacro:gripper.robotiq_gripper name="${tf_prefix}robotiq_2f_85"
+          prefix="${tf_prefix}"
+          parent="${parent_link}"
+          use_fake_hardware="false"
+          sim_ignition="true"
+        >
+          <origin xyz="${xyz}" rpy="${rpy}" />
+        </xacro:gripper.robotiq_gripper>
+      </xacro:if>
+      <xacro:if value="${type == 'GRP03'}">
+        <xacro:include filename="$(find robotiq_description)/urdf/robotiq_2f_140_macro.urdf.xacro"
+          ns="gripper" />
+        <xacro:gripper.robotiq_gripper name="${tf_prefix}robotiq_2f_140"
+          prefix="${tf_prefix}"
+          parent="${parent_link}"
+          use_fake_hardware="false"
+          sim_ignition="true"
+        >
+          <origin xyz="${xyz}" rpy="${rpy}" />
+        </xacro:gripper.robotiq_gripper>
+      </xacro:if>
       <xacro:if value="${index}">
         <xacro:load_componenet

Commit message: Made new tests
Signed-off-by: Jakub Delicat <jakub.delicat@husarion.com>

File: urdf/components.urdf.xacro (robot description, xacro)
@@ -23,5 +23,4 @@
       <xacro:property name="device_namespace" value="${component['device_namespace']}" scope="parent" />
       <xacro:if value="${type == 'CAM01'}">
-        <xacro:property name="camera_name" value="${component['name']}" scope="parent" />
         <xacro:include
           filename="$(find ros_components_description)/urdf/orbbec_astra.urdf.xacro"

File: urdf/orbbec_astra.urdf.xacro (robot description, xacro)
@@ -22,5 +22,5 @@
       <child link="${device_namespace}_orbbec_astra_link" />
     </joint>
-    <link name="${device_namespace}_orbbec_astra_link">
+    <link name="${device_namespace}_orbbec_astra">
       <visual>
         <origin xyz="0.0 0.0 0.0" rpy="0.0 0.0 0.0" />

File: urdf/slamtec_rplidar_a2.urdf.xacro (robot description, xacro)
@@ -82,5 +82,5 @@
       <!-- gpu_lidar has to be set, CPU lidar doesn't work in ignition -
       https://github.com/gazebosim/gz-sensors/issues/26 -->
-      <sensor type="gpu_lidar" name="${ns}${prefix}rplidar_a2_sensor">
+      <sensor type="gpu_lidar" name="${ns}${prefix}slamtec_rplidar_a2_sensor">
         <topic>${ns}${device_ns}scan</topic>
         <frame_id>${ns}${prefix}laser</frame_id>

File: urdf/slamtec_rplidar_a3.urdf.xacro (robot description, xacro)
@@ -59,5 +59,5 @@
       <!-- gpu_lidar has to be set, CPU lidar doesn't work in ignition -
       https://github.com/gazebosim/gz-sensors/issues/26 -->
-      <sensor type="gpu_lidar" name="${ns}${prefix}rplidar_a3_sensor">
+      <sensor type="gpu_lidar" name="${ns}${prefix}slamtec_rplidar_a3_sensor">
         <topic>${ns}${device_ns}scan</topic>
         <frame_id>${ns}${prefix}laser</frame_id>

File: urdf/slamtec_rplidar_s1.urdf.xacro (robot description, xacro)
@@ -66,5 +66,5 @@
       <!-- gpu_lidar has to be set, CPU lidar doesn't work in ignition -
       https://github.com/gazebosim/gz-sensors/issues/26 -->
-      <sensor type="gpu_lidar" name="${ns}${prefix}rplidar_s1_sensor">
+      <sensor type="gpu_lidar" name="${ns}${prefix}slamtec_rplidar_s1_sensor">
         <topic>${ns}${device_ns}scan</topic>
         <frame_id>${ns}${prefix}laser</frame_id>

File: urdf/slamtec_rplidar_s2.urdf.xacro (robot description, xacro)
@@ -59,5 +59,5 @@
       <!-- gpu_lidar has to be set, CPU lidar doesn't work in ignition -
       https://github.com/gazebosim/gz-sensors/issues/26 -->
-      <sensor type="gpu_lidar" name="${ns}${prefix}rplidar_s2_sensor">
+      <sensor type="gpu_lidar" name="${ns}${prefix}slamtec_rplidar_s2_sensor">
         <topic>${ns}${device_ns}scan</topic>
         <frame_id>${ns}${prefix}laser</frame_id>

File: urdf/slamtec_rplidar_s3.urdf.xacro (robot description, xacro)
@@ -59,5 +59,5 @@
       <!-- gpu_lidar has to be set, CPU lidar doesn't work in ignition -
       https://github.com/gazebosim/gz-sensors/issues/26 -->
-      <sensor type="gpu_lidar" name="${ns}${prefix}rplidar_s3_sensor">
+      <sensor type="gpu_lidar" name="${ns}${prefix}slamtec_rplidar_s3_sensor">
         <topic>${ns}${device_ns}scan</topic>
         <frame_id>${ns}${prefix}laser</frame_id>

Commit message: added  ouster os1 and os0

File: urdf/components.urdf.xacro (robot description, xacro)
@@ -60,15 +60,86 @@
         />
       </xacro:if>
+      <xacro:if value="${type == 'LDR10'}">
+        <xacro:include
+          filename="$(find ros_components_description)/urdf/ouster_os01.urdf.xacro"
+          ns="lidar"
+        />
+        <xacro:lidar.ouster_os01
+          parent_link="${parent_link}"
+          xyz="${xyz}"
+          rpy="${rpy}"
+          namespace="${robot_namespace}"
+          device_namespace="${device_namespace}"
+          model="os0_32"
+        />
+      </xacro:if>
+      <xacro:if value="${type == 'LDR11'}">
+        <xacro:include
+          filename="$(find ros_components_description)/urdf/ouster_os01.urdf.xacro"
+          ns="lidar"
+        />
+        <xacro:lidar.ouster_os01
+          parent_link="${parent_link}"
+          xyz="${xyz}"
+          rpy="${rpy}"
+          namespace="${robot_namespace}"
+          device_namespace="${device_namespace}"
+          model="os0_64"
+        />
+      </xacro:if>
+      <xacro:if value="${type == 'LDR12'}">
+        <xacro:include
+          filename="$(find ros_components_description)/urdf/ouster_os01.urdf.xacro"
+          ns="lidar"
+        />
+        <xacro:lidar.ouster_os01
+          parent_link="${parent_link}"
+          xyz="${xyz}"
+          rpy="${rpy}"
+          namespace="${robot_namespace}"
+          device_namespace="${device_namespace}"
+          model="os0_128"
+        />
+      </xacro:if>
       <xacro:if value="${type == 'LDR13'}">
         <xacro:include
-          filename="$(find ros_components_description)/urdf/ouster_os1_32.urdf.xacro"
-          ns="lidar"
-        />
-        <xacro:lidar.ouster_os1_32
-          parent_link="${parent_link}"
-          xyz="${xyz}"
-          rpy="${rpy}"
-          namespace="${robot_namespace}"
-          device_namespace="${device_namespace}"
+          filename="$(find ros_components_description)/urdf/ouster_os01.urdf.xacro"
+          ns="lidar"
+        />
+        <xacro:lidar.ouster_os01
+          parent_link="${parent_link}"
+          xyz="${xyz}"
+          rpy="${rpy}"
+          namespace="${robot_namespace}"
+          device_namespace="${device_namespace}"
+          model="os1_32"
+        />
+      </xacro:if>
+      <xacro:if value="${type == 'LDR14'}">
+        <xacro:include
+          filename="$(find ros_components_description)/urdf/ouster_os01.urdf.xacro"
+          ns="lidar"
+        />
+        <xacro:lidar.ouster_os01
+          parent_link="${parent_link}"
+          xyz="${xyz}"
+          rpy="${rpy}"
+          namespace="${robot_namespace}"
+          device_namespace="${device_namespace}"
+          model="os1_64"
+        />
+      </xacro:if>
+      <xacro:if value="${type == 'LDR15'}">
+        <xacro:include
+          filename="$(find ros_components_description)/urdf/ouster_os01.urdf.xacro"
+          ns="lidar"
+        />
+        <xacro:lidar.ouster_os01
+          parent_link="${parent_link}"
+          xyz="${xyz}"
+          rpy="${rpy}"
+          namespace="${robot_namespace}"
+          device_namespace="${device_namespace}"
+          model="os1_128"
         />
       </xacro:if>

File: urdf/ouster_os01.urdf.xacro (robot description, xacro)
@@ -1,8 +1,39 @@
 <?xml version="1.0"?>
 <robot xmlns:xacro="http://www.ros.org/wiki/xacro">
-    <xacro:macro name="ouster_os1_32"
+    <xacro:macro name="ouster_os01"
                params="parent_link xyz rpy
+                       model:=os1_32
                        namespace:=None
                        device_namespace:=None">
+    <xacro:if value="${model == 'os0_32'}">
+      <xacro:property name="vfov" value="${radians(90.0)}" scope="parent" />
+      <xacro:property name="lidar_range" value="50" scope="parent"/>
+      <xacro:property name="layers" value="32" scope="parent"/>
+    </xacro:if>
+    <xacro:if value="${model == 'os0_64'}">
+      <xacro:property name="vfov" value="${radians(90.0)}" scope="parent" />
+      <xacro:property name="lidar_range" value="50" scope="parent" />
+      <xacro:property name="layers" value="64" scope="parent" />
+    </xacro:if>
+    <xacro:if value="${model == 'os0_128'}">
+      <xacro:property name="vfov" value="${radians(90.0)}" scope="parent" />
+      <xacro:property name="lidar_range" value="50" scope="parent" />
+      <xacro:property name="layers" value="128" scope="parent" />
+    </xacro:if>
+    <xacro:if value="${model == 'os1_32'}">
+      <xacro:property name="vfov" value="${radians(45.0)}" scope="parent" />
+      <xacro:property name="lidar_range" value="120" scope="parent" />
+      <xacro:property name="layers" value="32" scope="parent" />
+    </xacro:if>
+    <xacro:if value="${model == 'os1_64'}">
+      <xacro:property name="vfov" value="${radians(45.0)}" scope="parent" />
+      <xacro:property name="lidar_range" value="120" scope="parent" />
+      <xacro:property name="layers" value="64" scope="parent" />
+    </xacro:if>
+    <xacro:if value="${model == 'os1_128'}">
+      <xacro:property name="vfov" value="${radians(45.0)}" scope="parent" />
+      <xacro:property name="lidar_range" value="120" scope="parent" />
+      <xacro:property name="layers" value="128" scope="parent" />
+    </xacro:if>
     <xacro:if value="${namespace == 'None'}">
       <xacro:property name="ns" value="" />
@@ -23,14 +54,14 @@
       <xacro:property name="prefix" value="${device_namespace}_" />
     </xacro:unless>
-    <joint name="${parent_link.rstrip('_link')}_to_${prefix}ouster_os1_32_joint" type="fixed">
+    <joint name="${parent_link.rstrip('_link')}_to_${prefix}ouster_${model}_joint" type="fixed">
       <origin xyz="${xyz}" rpy="${rpy}" />
       <parent link="${parent_link}" />
-      <child link="${prefix}ouster_os1_32_link" />
+      <child link="${prefix}ouster_${model}_link" />
     </joint>
-    <link name="${prefix}ouster_os1_32_link">
+    <link name="${prefix}ouster_${model}_link">
       <visual>
         <origin xyz="0.0 0.0 0.0" rpy="0.0 0.0 0.0" />
         <geometry>
-          <mesh filename="package://ros_components_description/meshes/ouster_os1_32.dae" />
+          <mesh filename="package://ros_components_description/meshes/ouster_os01.dae" />
         </geometry>
       </visual>
@@ -49,7 +80,7 @@
       </inertial>
     </link>
-    <joint name="${prefix}ouster_os1_32_to_${prefix}os_lidar_joint" type="fixed">
+    <joint name="${prefix}ouster_${model}_to_${prefix}os_lidar_joint" type="fixed">
       <origin xyz="0.0 0.0 0.03618" rpy="0.0 0.0 0.0" />
-      <parent link="${prefix}ouster_os1_32_link" />
+      <parent link="${prefix}ouster_${model}_link" />
       <child link="${prefix}os_lidar" />
     </joint>
@@ -58,5 +89,5 @@
       <!-- gpu_lidar has to be set, CPU lidar doesn't work in ignition -
       https://github.com/gazebosim/gz-sensors/issues/26 -->
-      <sensor type="gpu_lidar" name="${ns}${prefix}ouster_os1_32_sensor">
+      <sensor type="gpu_lidar" name="${ns}${prefix}ouster_${model}_sensor">
         <visualize>false</visualize>
         <ray>
@@ -69,13 +100,13 @@
             </horizontal>
             <vertical>
-              <samples>32</samples>
+              <samples>${layers}</samples>
               <resolution>1</resolution>
-              <min_angle>-${22.5/180.0*pi}</min_angle>
-              <max_angle>${22.5/180.0*pi}</max_angle>
+              <min_angle>${vfov/-2.0}</min_angle>
+              <max_angle>${vfov/2.0}</max_angle>
             </vertical>
           </scan>
           <range>
             <min>0.8</min>
-            <max>120.0</max>
+            <max>${lidar_range}</max>
             <resolution>0.003</resolution>
           </range>

Commit message: s unified mesh

File: urdf/components.urdf.xacro (robot description, xacro)
@@ -62,8 +62,8 @@
       <xacro:if value="${type == 'LDR10'}">
         <xacro:include
-          filename="$(find ros_components_description)/urdf/ouster_os01.urdf.xacro"
-          ns="lidar"
-        />
-        <xacro:lidar.ouster_os01
+          filename="$(find ros_components_description)/urdf/ouster.urdf.xacro"
+          ns="lidar"
+        />
+        <xacro:lidar.ouster
           parent_link="${parent_link}"
           xyz="${xyz}"
@@ -76,8 +76,8 @@
       <xacro:if value="${type == 'LDR11'}">
         <xacro:include
-          filename="$(find ros_components_description)/urdf/ouster_os01.urdf.xacro"
-          ns="lidar"
-        />
-        <xacro:lidar.ouster_os01
+          filename="$(find ros_components_description)/urdf/ouster.urdf.xacro"
+          ns="lidar"
+        />
+        <xacro:lidar.ouster
           parent_link="${parent_link}"
           xyz="${xyz}"
@@ -90,8 +90,8 @@
       <xacro:if value="${type == 'LDR12'}">
         <xacro:include
-          filename="$(find ros_components_description)/urdf/ouster_os01.urdf.xacro"
-          ns="lidar"
-        />
-        <xacro:lidar.ouster_os01
+          filename="$(find ros_components_description)/urdf/ouster.urdf.xacro"
+          ns="lidar"
+        />
+        <xacro:lidar.ouster
           parent_link="${parent_link}"
           xyz="${xyz}"
@@ -104,8 +104,8 @@
       <xacro:if value="${type == 'LDR13'}">
         <xacro:include
-          filename="$(find ros_components_description)/urdf/ouster_os01.urdf.xacro"
-          ns="lidar"
-        />
-        <xacro:lidar.ouster_os01
+          filename="$(find ros_components_description)/urdf/ouster.urdf.xacro"
+          ns="lidar"
+        />
+        <xacro:lidar.ouster
           parent_link="${parent_link}"
           xyz="${xyz}"
@@ -118,8 +118,8 @@
       <xacro:if value="${type == 'LDR14'}">
         <xacro:include
-          filename="$(find ros_components_description)/urdf/ouster_os01.urdf.xacro"
-          ns="lidar"
-        />
-        <xacro:lidar.ouster_os01
+          filename="$(find ros_components_description)/urdf/ouster.urdf.xacro"
+          ns="lidar"
+        />
+        <xacro:lidar.ouster
           parent_link="${parent_link}"
           xyz="${xyz}"
@@ -132,8 +132,8 @@
       <xacro:if value="${type == 'LDR15'}">
         <xacro:include
-          filename="$(find ros_components_description)/urdf/ouster_os01.urdf.xacro"
-          ns="lidar"
-        />
-        <xacro:lidar.ouster_os01
+          filename="$(find ros_components_description)/urdf/ouster.urdf.xacro"
+          ns="lidar"
+        />
+        <xacro:lidar.ouster
           parent_link="${parent_link}"
           xyz="${xyz}"

File: urdf/ouster.urdf.xacro (robot description, xacro)
@@ -1,5 +1,5 @@
 <?xml version="1.0"?>
 <robot xmlns:xacro="http://www.ros.org/wiki/xacro">
-    <xacro:macro name="ouster_os01"
+    <xacro:macro name="ouster"
                params="parent_link xyz rpy
                        model:=os1_32
@@ -10,4 +10,5 @@
       <xacro:property name="lidar_range" value="50" scope="parent"/>
       <xacro:property name="layers" value="32" scope="parent"/>
+      <xacro:property name="mesh" value="ouster_os01" scope="parent"/>
     </xacro:if>
     <xacro:if value="${model == 'os0_64'}">
@@ -15,4 +16,5 @@
       <xacro:property name="lidar_range" value="50" scope="parent" />
       <xacro:property name="layers" value="64" scope="parent" />
+      <xacro:property name="mesh" value="ouster_os01" scope="parent"/>
     </xacro:if>
     <xacro:if value="${model == 'os0_128'}">
@@ -20,4 +22,5 @@
       <xacro:property name="lidar_range" value="50" scope="parent" />
       <xacro:property name="layers" value="128" scope="parent" />
+      <xacro:property name="mesh" value="ouster_os01" scope="parent"/>
     </xacro:if>
     <xacro:if value="${model == 'os1_32'}">
@@ -25,4 +28,5 @@
       <xacro:property name="lidar_range" value="120" scope="parent" />
       <xacro:property name="layers" value="32" scope="parent" />
+      <xacro:property name="mesh" value="ouster_os01" scope="parent"/>
     </xacro:if>
     <xacro:if value="${model == 'os1_64'}">
@@ -30,4 +34,5 @@
       <xacro:property name="lidar_range" value="120" scope="parent" />
       <xacro:property name="layers" value="64" scope="parent" />
+      <xacro:property name="mesh" value="ouster_os01" scope="parent"/>
     </xacro:if>
     <xacro:if value="${model == 'os1_128'}">
@@ -35,4 +40,5 @@
       <xacro:property name="lidar_range" value="120" scope="parent" />
       <xacro:property name="layers" value="128" scope="parent" />
+      <xacro:property name="mesh" value="ouster_os01" scope="parent"/>
     </xacro:if>
     <xacro:if value="${namespace == 'None'}">
@@ -63,5 +69,5 @@
         <origin xyz="0.0 0.0 0.0" rpy="0.0 0.0 0.0" />
         <geometry>
-          <mesh filename="package://ros_components_description/meshes/ouster_os01.dae" />
+          <mesh filename="package://ros_components_description/meshes/${mesh}.dae" />
         </geometry>
       </visual>
