Commit message: Added zed
Signed-off-by: Jakub Delicat <jakub.delicat@husarion.com>

File: urdf/components.urdf.xacro (robot description, xacro)
@@ -34,4 +34,17 @@
         />
       </xacro:if>
+      <xacro:if value="${type == 'CAM03'}">
+        <xacro:include
+          filename="$(find ros_components_description)/urdf/stereolabs_zed.urdf.xacro"
+          ns="camera" />
+        <xacro:camera.zed_camera
+          parent_link="${parent_link}"
+          xyz="${xyz}"
+          rpy="${rpy}"
+          model="zed2"
+          namespace="${robot_namespace}"
+          device_namespace="${device_namespace}"
+        />
+      </xacro:if>
       <xacro:if value="${type == 'LDR01'}">
         <xacro:include

File: urdf/stereolabs_zed.urdf.xacro (robot description, xacro)
@@ -107,8 +107,8 @@
     <!-- Artificially Created Camera Center -->
     <link name="${device_namespace}_center_optical_frame" />
-    <joint name="${device_namespace}_center_joint" type="fixed">
+    <joint name="${device_namespace}_artificial_center_joint" type="fixed">
       <parent link="${device_namespace}_center" />
       <child link="${device_namespace}_center_optical_frame" />
-      <origin xyz="0.01 0 0" rpy="0 0 0" />
+      <origin xyz="0.05 0 0" rpy="0 0 0" />
     </joint>
     <!-- Left Camera -->
@@ -187,5 +187,5 @@
       <sensor type="depth_camera" name="${ns}${device_namespace}_stereolabs_zed_depth">
         <always_on>true</always_on>
-        <update_rate>30.0</update_rate>
+        <update_rate>10.0</update_rate>
         <topic>${ns}${device_namespace}/zed_node/depth</topic>
         <visualize>false</visualize>

Commit message: ROS 2 ouster os1 os0 (#47)
* Fixed prefix

Signed-off-by: Jakub Delicat <jakub.delicat@husarion.com>

* Added launches and gz mappings

Signed-off-by: Jakub Delicat <jakub.delicat@husarion.com>

* update launches

Signed-off-by: Jakub Delicat <jakub.delicat@husarion.com>

* fixed astra

Signed-off-by: Jakub Delicat <jakub.delicat@husarion.com>

* removed print

Signed-off-by: Jakub Delicat <jakub.delicat@husarion.com>

* Fixed unused file

Signed-off-by: Jakub Delicat <jakub.delicat@husarion.com>

* renamed files

Signed-off-by: Jakub Delicat <jakub.delicat@husarion.com>

* Added ur

Signed-off-by: Jakub Delicat <jakub.delicat@husarion.com>

* added kinova

Signed-off-by: Jakub Delicat <jakub.delicat@husarion.com>

* split 6dof and 7dof

Signed-off-by: Jakub Delicat <jakub.delicat@husarion.com>

* Added rootiq

Signed-off-by: Jakub Delicat <jakub.delicat@husarion.com>

* Added suggestion

Signed-off-by: Jakub Delicat <jakub.delicat@husarion.com>

* simplfied urfd | removed use_gpu | removed simulation-engine

Signed-off-by: Jakub Delicat <jakub.delicat@husarion.com>

* simplfied urfd | removed use_gpu | removed simulation-engine

Signed-off-by: Jakub Delicat <jakub.delicat@husarion.com>

* applied new changes to ur

Signed-off-by: Jakub Delicat <jakub.delicat@husarion.com>

* removed simulation-engine from s3 | fix with no namespace

Signed-off-by: Jakub Delicat <jakub.delicat@husarion.com>

* fixed namespaced ros2_control

Signed-off-by: Jakub Delicat <jakub.delicat@husarion.com>

* Suggestions

* add

* workflow simplify

* Removed unnecessary topic form realsense

Signed-off-by: Jakub Delicat <jakub.delicat@husarion.com>

* Made new tests

Signed-off-by: Jakub Delicat <jakub.delicat@husarion.com>

* fixed astra

Signed-off-by: Jakub Delicat <jakub.delicat@husarion.com>

* applied tests

Signed-off-by: Jakub Delicat <jakub.delicat@husarion.com>

* Added comment about GRP03

Signed-off-by: Jakub Delicat <jakub.delicat@husarion.com>

* added  ouster os1 and os0

* s unified mesh

* Suggestion and namespace fix

Signed-off-by: Jakub Delicat <jakub.delicat@husarion.com>

---------

Signed-off-by: Jakub Delicat <jakub.delicat@husarion.com>
Co-authored-by: rafal-gorecki <rafal.gorecki@husarion.com>
Co-authored-by: rafal-gorecki <126687345+rafal-gorecki@users.noreply.github.com>

File: urdf/components.urdf.xacro (robot description, xacro)
@@ -21,5 +21,6 @@
       <xacro:property name="xyz" value="${component['xyz']}" scope="parent" />
       <xacro:property name="rpy" value="${component['rpy']}" scope="parent" />
-      <xacro:property name="device_namespace" value="${component['device_namespace']}" scope="parent" />
+      <xacro:property name="device_namespace" value="${component['device_namespace']}"
+        scope="parent" />
       <xacro:if value="${type == 'CAM01'}">
         <xacro:include
@@ -60,15 +61,25 @@
         />
       </xacro:if>
-      <xacro:if value="${type == 'LDR13'}">
-        <xacro:include
-          filename="$(find ros_components_description)/urdf/ouster_os1_32.urdf.xacro"
-          ns="lidar"
-        />
-        <xacro:lidar.ouster_os1_32
-          parent_link="${parent_link}"
-          xyz="${xyz}"
-          rpy="${rpy}"
-          namespace="${robot_namespace}"
-          device_namespace="${device_namespace}"
+      <xacro:property name="ouster_models_dict"
+        value="${dict ([
+        ('LDR10', 'os0_32'),
+        ('LDR11', 'os0_64'),
+        ('LDR12', 'os0_128'),
+        ('LDR13', 'os1_32'),
+        ('LDR14', 'os1_64'),
+        ('LDR15', 'os1_128')
+      ])}" />
+      <xacro:if value="${type in ouster_models_dict}">
+        <xacro:include
+          filename="$(find ros_components_description)/urdf/ouster.urdf.xacro"
+          ns="lidar"
+        />
+        <xacro:lidar.ouster
+          parent_link="${parent_link}"
+          xyz="${xyz}"
+          rpy="${rpy}"
+          namespace="${robot_namespace}"
+          device_namespace="${device_namespace}"
+          model="${ouster_models_dict[type]}"
         />
       </xacro:if>

File: urdf/ouster.urdf.xacro (robot description, xacro)
@@ -1,8 +1,45 @@
 <?xml version="1.0"?>
 <robot xmlns:xacro="http://www.ros.org/wiki/xacro">
-    <xacro:macro name="ouster_os1_32"
+    <xacro:macro name="ouster"
                params="parent_link xyz rpy
+                       model:=os1_32
                        namespace:=None
                        device_namespace:=None">
+    <xacro:if value="${model == 'os0_32'}">
+      <xacro:property name="vfov" value="${radians(90.0)}" scope="parent" />
+      <xacro:property name="lidar_range" value="50" scope="parent"/>
+      <xacro:property name="layers" value="32" scope="parent"/>
+      <xacro:property name="mesh" value="ouster_os01" scope="parent"/>
+    </xacro:if>
+    <xacro:if value="${model == 'os0_64'}">
+      <xacro:property name="vfov" value="${radians(90.0)}" scope="parent" />
+      <xacro:property name="lidar_range" value="50" scope="parent" />
+      <xacro:property name="layers" value="64" scope="parent" />
+      <xacro:property name="mesh" value="ouster_os01" scope="parent"/>
+    </xacro:if>
+    <xacro:if value="${model == 'os0_128'}">
+      <xacro:property name="vfov" value="${radians(90.0)}" scope="parent" />
+      <xacro:property name="lidar_range" value="50" scope="parent" />
+      <xacro:property name="layers" value="128" scope="parent" />
+      <xacro:property name="mesh" value="ouster_os01" scope="parent"/>
+    </xacro:if>
+    <xacro:if value="${model == 'os1_32'}">
+      <xacro:property name="vfov" value="${radians(45.0)}" scope="parent" />
+      <xacro:property name="lidar_range" value="120" scope="parent" />
+      <xacro:property name="layers" value="32" scope="parent" />
+      <xacro:property name="mesh" value="ouster_os01" scope="parent"/>
+    </xacro:if>
+    <xacro:if value="${model == 'os1_64'}">
+      <xacro:property name="vfov" value="${radians(45.0)}" scope="parent" />
+      <xacro:property name="lidar_range" value="120" scope="parent" />
+      <xacro:property name="layers" value="64" scope="parent" />
+      <xacro:property name="mesh" value="ouster_os01" scope="parent"/>
+    </xacro:if>
+    <xacro:if value="${model == 'os1_128'}">
+      <xacro:property name="vfov" value="${radians(45.0)}" scope="parent" />
+      <xacro:property name="lidar_range" value="120" scope="parent" />
+      <xacro:property name="layers" value="128" scope="parent" />
+      <xacro:property name="mesh" value="ouster_os01" scope="parent"/>
+    </xacro:if>
     <xacro:if value="${namespace == 'None'}">
       <xacro:property name="ns" value="" />
@@ -23,14 +60,14 @@
       <xacro:property name="prefix" value="${device_namespace}_" />
     </xacro:unless>
-    <joint name="${parent_link.rstrip('_link')}_to_${prefix}ouster_os1_32_joint" type="fixed">
+    <joint name="${parent_link.rstrip('_link')}_to_${prefix}ouster_${model}_joint" type="fixed">
       <origin xyz="${xyz}" rpy="${rpy}" />
       <parent link="${parent_link}" />
-      <child link="${prefix}ouster_os1_32_link" />
+      <child link="${prefix}ouster_${model}_link" />
     </joint>
-    <link name="${prefix}ouster_os1_32_link">
+    <link name="${prefix}ouster_${model}_link">
       <visual>
         <origin xyz="0.0 0.0 0.0" rpy="0.0 0.0 0.0" />
         <geometry>
-          <mesh filename="package://ros_components_description/meshes/ouster_os1_32.dae" />
+          <mesh filename="package://ros_components_description/meshes/${mesh}.dae" />
         </geometry>
       </visual>
@@ -49,7 +86,7 @@
       </inertial>
     </link>
-    <joint name="${prefix}ouster_os1_32_to_${prefix}os_lidar_joint" type="fixed">
+    <joint name="${prefix}ouster_${model}_to_${prefix}os_lidar_joint" type="fixed">
       <origin xyz="0.0 0.0 0.03618" rpy="0.0 0.0 0.0" />
-      <parent link="${prefix}ouster_os1_32_link" />
+      <parent link="${prefix}ouster_${model}_link" />
       <child link="${prefix}os_lidar" />
     </joint>
@@ -58,5 +95,5 @@
       <!-- gpu_lidar has to be set, CPU lidar doesn't work in ignition -
       https://github.com/gazebosim/gz-sensors/issues/26 -->
-      <sensor type="gpu_lidar" name="${ns}${prefix}ouster_os1_32_sensor">
+      <sensor type="gpu_lidar" name="${ns}${prefix}ouster_${model}_sensor">
         <visualize>false</visualize>
         <ray>
@@ -69,13 +106,13 @@
             </horizontal>
             <vertical>
-              <samples>32</samples>
+              <samples>${layers}</samples>
               <resolution>1</resolution>
-              <min_angle>-${22.5/180.0*pi}</min_angle>
-              <max_angle>${22.5/180.0*pi}</max_angle>
+              <min_angle>${vfov/-2.0}</min_angle>
+              <max_angle>${vfov/2.0}</max_angle>
             </vertical>
           </scan>
           <range>
             <min>0.8</min>
-            <max>120.0</max>
+            <max>${lidar_range}</max>
             <resolution>0.003</resolution>
           </range>

Commit message: No namespaces TF fix (#49)
* No namespaces fix

Signed-off-by: Jakub Delicat <jakub.delicat@husarion.com>

* Add lazy, fix and simplify orbbec_astra, remove <ros> from <sensor>

* Delete unused arg

* Rebase branch

* revert astra resolution

Signed-off-by: Jakub Delicat <jakub.delicat@husarion.com>

* without namespace working

Signed-off-by: Jakub Delicat <jakub.delicat@husarion.com>

---------

Signed-off-by: Jakub Delicat <jakub.delicat@husarion.com>
Co-authored-by: rafal-gorecki <rafal.gorecki@husarion.com>

File: urdf/components.urdf.xacro (robot description, xacro)
@@ -23,4 +23,10 @@
       <xacro:property name="device_namespace" value="${component['device_namespace']}"
         scope="parent" />
+        <xacro:if value="${robot_namespace == ''}">
+          <xacro:property name="ns" value="None" scope="parent" />
+        </xacro:if>
+        <xacro:unless value="${robot_namespace == ''}">
+          <xacro:property name="ns" value="${robot_namespace}" scope="parent" />
+        </xacro:unless>
       <xacro:if value="${type == 'CAM01'}">
         <xacro:include
@@ -31,5 +37,5 @@
           xyz="${xyz}"
           rpy="${rpy}"
-          namespace="${robot_namespace}"
+          namespace="${ns}"
           device_namespace="${device_namespace}"
         />
@@ -44,5 +50,5 @@
           xyz="${xyz}"
           rpy="${rpy}"
-          namespace="${robot_namespace}"
+          namespace="${ns}"
           device_namespace="${device_namespace}"
         />
@@ -57,5 +63,5 @@
           xyz="${xyz}"
           rpy="${rpy}"
-          namespace="${robot_namespace}"
+          namespace="${ns}"
           device_namespace="${device_namespace}"
         />
@@ -79,5 +85,5 @@
           xyz="${xyz}"
           rpy="${rpy}"
-          namespace="${robot_namespace}"
+          namespace="${ns}"
           device_namespace="${device_namespace}"
           model="${ouster_models_dict[type]}"
@@ -93,5 +99,5 @@
           xyz="${xyz}"
           rpy="${rpy}"
-          namespace="${robot_namespace}"
+          namespace="${ns}"
           device_namespace="${device_namespace}"
         />
@@ -132,5 +138,5 @@
           xyz="${xyz}"
           rpy="${rpy}"
-          namespace="${robot_namespace}"
+          namespace="${ns}"
           device_namespace="${device_namespace}"
           kinova_type="gen3"
@@ -149,5 +155,5 @@
           xyz="${xyz}"
           rpy="${rpy}"
-          namespace="${robot_namespace}"
+          namespace="${ns}"
           device_namespace="${device_namespace}"
           kinova_type="gen3"
@@ -166,5 +172,5 @@
           xyz="${xyz}"
           rpy="${rpy}"
-          namespace="${robot_namespace}"
+          namespace="${ns}"
           device_namespace="${device_namespace}"
           kinova_type="gen3"
@@ -183,5 +189,5 @@
           xyz="${xyz}"
           rpy="${rpy}"
-          namespace="${robot_namespace}"
+          namespace="${ns}"
           kinova_type="gen3"
           dof="7"
@@ -198,5 +204,5 @@
           xyz="${xyz}"
           rpy="${rpy}"
-          namespace="${robot_namespace}"
+          namespace="${ns}"
           device_namespace="${device_namespace}"
           robotiq_type="2f_85"

File: urdf/intel_realsense_d435.urdf.xacro (robot description, xacro)
@@ -164,7 +164,4 @@
           <far>300.0</far>
         </clip>
-        <ros>
-          <namespace>${ns}${device_namespace}</namespace>
-        </ros>
       </sensor>
       <sensor type="depth_camera" name="${ns}${device_namespace}_intel_realsense_d435_depth">
@@ -191,7 +188,4 @@
           </noise>
         </camera>
-        <ros>
-          <namespace>${ns}${device_namespace}</namespace>
-        </ros>
       </sensor>
     </gazebo>

File: urdf/kinova.urdf.xacro (robot description, xacro)
@@ -172,7 +172,4 @@
           <topic>${ns}${device_namespace}/wrist_mounted_camera</topic>
           <enable_metrics>false</enable_metrics>
-          <ros>
-            <namespace>${ns}${device_namespace}</namespace>
-          </ros>
         </sensor>
       </gazebo>

File: urdf/orbbec_astra.urdf.xacro (robot description, xacro)
@@ -82,5 +82,5 @@
         <topic>${ns}${device_namespace}/color/image_raw</topic>
         <visualize>false</visualize>
-        <ignition_frame_id>${device_namespace}_color_optical_frame</ignition_frame_id>
+        <ignition_frame_id>${ns}${device_namespace}_color_optical_frame</ignition_frame_id>
         <horizontal_fov>${60.0/180.0*pi}</horizontal_fov>
         <image>
@@ -92,7 +92,4 @@
           <far>8.0</far>
         </clip>
-        <ros>
-          <namespace>${ns}${device_namespace}</namespace>
-        </ros>
       </sensor>
       <sensor type="depth_camera" name="${ns}${device_namespace}_orbbec_astra_depth">
@@ -101,5 +98,5 @@
         <topic>${ns}${device_namespace}/depth/image_raw</topic>
         <visualize>false</visualize>
-        <ignition_frame_id>${device_namespace}_depth_optical_frame</ignition_frame_id>
+        <ignition_frame_id>${ns}${device_namespace}_depth_optical_frame</ignition_frame_id>
         <camera>
           <horizontal_fov>${60.0/180.0*pi}</horizontal_fov>
@@ -118,7 +115,4 @@
           </noise>
         </camera>
-        <ros>
-          <namespace>${ns}${device_namespace}</namespace>
-        </ros>
       </sensor>
     </gazebo>

File: urdf/ouster.urdf.xacro (robot description, xacro)
@@ -128,7 +128,4 @@
         <ignition_frame_id>${ns}${prefix}os_lidar</ignition_frame_id>
         <always_on>true</always_on>
-        <ros>
-          <namespace>${ns}${device_ns}</namespace>
-        </ros>
       </sensor>
     </gazebo>

File: urdf/slamtec_rplidar_a2.urdf.xacro (robot description, xacro)
@@ -109,7 +109,4 @@
         <always_on>true</always_on>
         <visualize>false</visualize>
-        <ros>
-          <namespace>${ns}${device_ns}</namespace>
-        </ros>
       </sensor>
     </gazebo>

File: urdf/slamtec_rplidar_a3.urdf.xacro (robot description, xacro)
@@ -87,7 +87,4 @@
         <always_on>true</always_on>
         <visualize>false</visualize>
-        <ros>
-          <namespace>${ns}${device_ns}</namespace>
-        </ros>
       </sensor>
     </gazebo>

File: urdf/slamtec_rplidar_s1.urdf.xacro (robot description, xacro)
@@ -93,7 +93,4 @@
         <always_on>true</always_on>
         <visualize>false</visualize>
-        <ros>
-          <namespace>${ns}${device_ns}</namespace>
-        </ros>
       </sensor>
     </gazebo>

File: urdf/slamtec_rplidar_s2.urdf.xacro (robot description, xacro)
@@ -86,7 +86,4 @@
         <always_on>1</always_on>
         <visualize>false</visualize>
-        <ros>
-          <namespace>${ns}${device_ns}</namespace>
-        </ros>
       </sensor>
     </gazebo>

File: urdf/slamtec_rplidar_s3.urdf.xacro (robot description, xacro)
@@ -86,7 +86,4 @@
         <always_on>1</always_on>
         <visualize>false</visualize>
-        <ros>
-          <namespace>${ns}${device_ns}</namespace>
-        </ros>
       </sensor>
     </gazebo>

File: urdf/stereolabs_zed.urdf.xacro (robot description, xacro)
@@ -181,7 +181,4 @@
           </clip>
         </camera>
-        <ros>
-          <namespace>${ns}</namespace>
-        </ros>
       </sensor>
       <sensor type="depth_camera" name="${ns}${device_namespace}_stereolabs_zed_depth">
@@ -207,7 +204,4 @@
           </noise>
         </camera>
-        <ros>
-          <namespace>${ns}${device_namespace}</namespace>
-        </ros>
       </sensor>
     </gazebo>

File: urdf/velodyne_puck.urdf.xacro (robot description, xacro)
@@ -92,7 +92,4 @@
         <ignition_frame_id>${ns}${prefix}velodyne</ignition_frame_id>
         <always_on>true</always_on>
-        <ros>
-          <namespace>${ns}${device_ns}</namespace>
-        </ros>
       </sensor>
     </gazebo>

Commit message: ROS 2 ZED Gazebo Components fix (#53)
* No namespaces fix

Signed-off-by: Jakub Delicat <jakub.delicat@husarion.com>

* Add lazy, fix and simplify orbbec_astra, remove <ros> from <sensor>

* Delete unused arg

* Rebase branch

* WIP zed

Signed-off-by: Jakub Delicat <jakub.delicat@husarion.com>

* WIP Zed

Signed-off-by: Jakub Delicat <jakub.delicat@husarion.com>

* revert astra resolution

Signed-off-by: Jakub Delicat <jakub.delicat@husarion.com>

* without namespace working

Signed-off-by: Jakub Delicat <jakub.delicat@husarion.com>

* Added zed

Signed-off-by: Jakub Delicat <jakub.delicat@husarion.com>

* Tests

Signed-off-by: Jakub Delicat <jakub.delicat@husarion.com>

* added CR

Signed-off-by: Jakub Delicat <jakub.delicat@husarion.com>

---------

Signed-off-by: Jakub Delicat <jakub.delicat@husarion.com>
Co-authored-by: rafal-gorecki <rafal.gorecki@husarion.com>

File: urdf/components.urdf.xacro (robot description, xacro)
@@ -41,4 +41,23 @@
         />
       </xacro:if>
+      <xacro:property name="zed_models_dict"
+        value="${dict ([
+        ('CAM03', 'zed2'),
+        ('CAM04', 'zed2i'),
+        ('CAM06', 'zedx'),
+        ])}" />
+        <xacro:if value="${type in zed_models_dict}">
+        <xacro:include
+          filename="$(find ros_components_description)/urdf/stereolabs_zed.urdf.xacro"
+          ns="camera" />
+        <xacro:camera.zed_camera
+          parent_link="${parent_link}"
+          xyz="${xyz}"
+          rpy="${rpy}"
+          namespace="${ns}"
+          device_namespace="${device_namespace}"
+          model="${zed_models_dict[type]}"
+        />
+      </xacro:if>
       <xacro:if value="${type == 'LDR01'}">
         <xacro:include

File: urdf/stereolabs_zed.urdf.xacro (robot description, xacro)
@@ -1,4 +1,5 @@
 <?xml version="1.0"?>
 <!--
+// Copyright 2024 Husarion sp. z o.o.
 // Copyright 2022 Stereolabs
 //
@@ -100,5 +101,5 @@
       </collision>
     </link>
-    <joint name="${device_namespace}_center_joint" type="fixed">
+    <joint name="${device_namespace}_camera_center_joint" type="fixed">
       <parent link="${device_namespace}_link" />
       <child link="${device_namespace}_center" />
