Commit message: Rplidar-merge (#52)
* Rplidar-merge

* Fix urdf

File: urdf/components.urdf.xacro (robot description, xacro)
@@ -60,28 +60,21 @@
         />
       </xacro:if>
-      <xacro:if value="${type == 'LDR01'}">
-        <xacro:include
-          filename="$(find ros_components_description)/urdf/slamtec_rplidar_s1.urdf.xacro"
+      <xacro:property name="rplidar_models_dict"
+        value="${dict ([
+        ('LDR01', 's1'),
+        ('LDR06', 's3'),
+      ])}" />
+      <xacro:if value="${type in rplidar_models_dict}">
+        <xacro:include
+          filename="$(find ros_components_description)/urdf/slamtec_rplidar.urdf.xacro"
           ns="lidar"
         />
-        <xacro:lidar.slamtec_rplidar_s1
-          parent_link="${parent_link}"
-          xyz="${xyz}"
-          rpy="${rpy}"
-          namespace="${ns}"
-          device_namespace="${device_namespace}"
-        />
-      </xacro:if>
-      <xacro:if value="${type == 'LDR06'}">
-        <xacro:include
-          filename="$(find ros_components_description)/urdf/slamtec_rplidar_s3.urdf.xacro"
-          ns="lidar"
-        />
-        <xacro:lidar.slamtec_rplidar_s3
-          parent_link="${parent_link}"
-          xyz="${xyz}"
-          rpy="${rpy}"
-          namespace="${ns}"
-          device_namespace="${device_namespace}"
+        <xacro:lidar.slamtec_rplidar
+          parent_link="${parent_link}"
+          xyz="${xyz}"
+          rpy="${rpy}"
+          namespace="${ns}"
+          device_namespace="${device_namespace}"
+          model="${rplidar_models_dict[type]}"
         />
       </xacro:if>

File: urdf/intel_realsense_d435.urdf.xacro (robot description, xacro)
@@ -33,7 +33,7 @@
     <xacro:property name="d435_cam_depth_to_infra2_offset" value="-0.050" />
     <xacro:property name="d435_cam_depth_to_color_offset" value="0.015" />
-    <!-- The following values model the aluminum peripherial case for the
+    <!-- The following values model the aluminum peripheral case for the
       D435 camera, with the camera joint represented by the actual
-      peripherial camera tripod mount -->
+      peripheral camera tripod mount -->
     <xacro:property name="d435_cam_width" value="0.090" />
     <xacro:property name="d435_cam_height" value="0.025" />
@@ -47,5 +47,5 @@
     <xacro:property name="d435_mesh_x_offset"
       value="${d435_cam_mount_from_center_offset-d435_glass_to_front-d435_zero_depth_to_glass}" />
-    <!-- The following offset is relative the the physical D435 camera peripherial
+    <!-- The following offset is relative the the physical D435 camera peripheral
       camera tripod mount -->
     <xacro:property name="d435_cam_depth_px" value="${d435_cam_mount_from_center_offset}" />

Commit message: Add antenna (#50)
* Add pre commit

* Add external antenna

* Rename extenal antena -> teltonika

* Set GPS uptade rate to 1Hz

* Add ns to tf frame

* Update name

* Mounting point

File: urdf/components.urdf.xacro (robot description, xacro)
@@ -23,10 +23,22 @@
       <xacro:property name="device_namespace" value="${component['device_namespace']}"
         scope="parent" />
-        <xacro:if value="${robot_namespace == ''}">
-          <xacro:property name="ns" value="None" scope="parent" />
-        </xacro:if>
-        <xacro:unless value="${robot_namespace == ''}">
-          <xacro:property name="ns" value="${robot_namespace}" scope="parent" />
-        </xacro:unless>
+      <xacro:if value="${robot_namespace == ''}">
+        <xacro:property name="ns" value="None" scope="parent" />
+      </xacro:if>
+      <xacro:unless value="${robot_namespace == ''}">
+        <xacro:property name="ns" value="${robot_namespace}" scope="parent" />
+      </xacro:unless>
+      <xacro:if value="${type == 'ANT02'}">
+        <xacro:include
+          filename="$(find ros_components_description)/urdf/teltonika_003R-00253.urdf.xacro"
+          ns="teltonika" />
+        <xacro:teltonika.teltonika_003R-00253
+          parent_link="${parent_link}"
+          xyz="${xyz}"
+          rpy="${rpy}"
+          namespace="${ns}"
+          device_namespace="${device_namespace}"
+        />
+      </xacro:if>
       <xacro:if value="${type == 'CAM01'}">
         <xacro:include
