Commit message: Fixes to noise model of S2

File: urdf/slamtec_rplidar.urdf.xacro (robot description, xacro)
@@ -55,5 +55,5 @@
       <xacro:property name="dist_max" value="30.0" />
       <xacro:property name="dist_res" value="0.013" />
-      <xacro:property name="std_dev" value="0.03" />
+      <xacro:property name="std_dev" value="0.003" />
       <xacro:property name="mesh" value="slamtec_rplidar_s2.dae" />
       <xacro:property name="collision">
