Commit message: Suggestions

File: test/component.urdf.xacro (robot description, xacro)
@@ -9,6 +9,4 @@
     <xacro:husarion_components.create_components
       components_config_path="${components_config_path_property}"
-      use_gpu="True"
-      simulation_engine="ignition-gazebo"
       namespace="None"
     />

File: urdf/intel_realsense_d435.urdf.xacro (robot description, xacro)
@@ -19,10 +19,8 @@
   <xacro:macro name="intel_realsense_d435"
     params="parent_link xyz rpy
-            tf_prefix:=None
-            name:=camera
             topic:=camera
             use_nominal_extrinsics:=false
             namespace:=None
-            simulation_engine:=ignition-gazebo">
+            device_namespace:=camera">
     <xacro:if value="${namespace == 'None'}">
       <xacro:property name="ns" value="" />
@@ -30,10 +28,4 @@
     <xacro:unless value="${namespace == 'None'}">
         <xacro:property name="ns" value="${namespace}/" />
-    </xacro:unless>
-    <xacro:if value="${tf_prefix == 'None'}">
-      <xacro:property name="prefix" value="" />
-    </xacro:if>
-    <xacro:unless value="${tf_prefix == 'None'}">
-      <xacro:property name="prefix" value="${tf_prefix}_" />
     </xacro:unless>
     <!-- The following values are approximate, and the camera node
@@ -63,17 +55,17 @@
     <xacro:property name="d435_cam_depth_pz" value="${d435_cam_height/2}" />
     <!-- camera body, with origin at bottom screw mount -->
-    <joint name="${parent_link.rstrip('_link')}_to_${prefix}${name}_bottom_screw_joint" type="fixed">
+    <joint name="${parent_link.rstrip('_link')}_to_${device_namespace}_bottom_screw_joint" type="fixed">
       <origin xyz="${xyz}" rpy="${rpy}" />
       <parent link="${parent_link}" />
-      <child link="${prefix}${name}_bottom_screw_frame" />
+      <child link="${device_namespace}_bottom_screw_frame" />
     </joint>
-    <link name="${prefix}${name}_bottom_screw_frame" />
-    <joint name="${prefix}${name}_bottom_screw_to_${prefix}${name}_joint" type="fixed">
+    <link name="${device_namespace}_bottom_screw_frame" />
+    <joint name="${device_namespace}_bottom_screw_to_${device_namespace}_joint" type="fixed">
       <origin xyz="${d435_mesh_x_offset} ${d435_cam_depth_py} ${d435_cam_depth_pz}"
         rpy="0.0 0.0 0.0" />
-      <parent link="${prefix}${name}_bottom_screw_frame" />
-      <child link="${prefix}${name}_link" />
+      <parent link="${device_namespace}_bottom_screw_frame" />
+      <child link="${device_namespace}_link" />
     </joint>
-    <link name="${prefix}${name}_link">
+    <link name="${device_namespace}_link">
       <visual>
         <origin xyz="0.0 0.0 0.0" rpy="0.0 0.0 0.0" />
@@ -101,110 +93,108 @@
     <xacro:if value="${use_nominal_extrinsics}">
       <!-- camera depth joints and links -->
-      <joint name="${prefix}${name}_to_${prefix}${name}_depth_joint" type="fixed">
+      <joint name="${device_namespace}_to_${device_namespace}_depth_joint" type="fixed">
         <origin xyz="0.0 0.0 0.0" rpy="0.0 0.0 0.0" />
-        <parent link="${prefix}${name}_link" />
-        <child link="${prefix}${name}_depth_frame" />
-      </joint>
-      <link name="${prefix}${name}_depth_frame" />
-      <joint name="${prefix}${name}_depth_to_${prefix}${name}_depth_optical_joint" type="fixed">
-        <origin xyz="0.0 0.0 0.0" rpy="${-pi/2.0} 0.0 ${-pi/2.0}" />
-        <parent link="${prefix}${name}_depth_frame" />
-        <child link="${prefix}${name}_depth_optical_frame" />
-      </joint>
-      <link name="${prefix}${name}_depth_optical_frame" />
+        <parent link="${device_namespace}_link" />
+        <child link="${device_namespace}_depth_frame" />
+      </joint>
+      <link name="${device_namespace}_depth_frame" />
+      <joint name="${device_namespace}_depth_to_${device_namespace}_depth_optical_joint" type="fixed">
+        <origin xyz="0.0 0.0 0.0" rpy="${-pi/2.0} 0.0 ${-pi/2.0}" />
+        <parent link="${device_namespace}_depth_frame" />
+        <child link="${device_namespace}_depth_optical_frame" />
+      </joint>
+      <link name="${device_namespace}_depth_optical_frame" />
       <!-- camera left IR joints and links -->
-      <joint name="${prefix}${name}_to_${prefix}${name}_infra1_joint" type="fixed">
+      <joint name="${device_namespace}_to_${device_namespace}_infra1_joint" type="fixed">
         <origin xyz="0.0 ${d435_cam_depth_to_infra1_offset} 0.0" rpy="0.0 0.0 0.0" />
-        <parent link="${prefix}${name}_link" />
-        <child link="${prefix}${name}_infra1_frame" />
-      </joint>
-      <link name="${prefix}${name}_infra1_frame" />
-      <joint name="${prefix}${name}_infra1_to_${prefix}${name}_infra1_optical_joint" type="fixed">
-        <origin xyz="0.0 0.0 0.0" rpy="${-pi/2.0} 0.0 ${-pi/2.0}" />
-        <parent link="${prefix}${name}_infra1_frame" />
-        <child link="${prefix}${name}_infra1_optical_frame" />
-      </joint>
-      <link name="${prefix}${name}_infra1_optical_frame" />
+        <parent link="${device_namespace}_link" />
+        <child link="${device_namespace}_infra1_frame" />
+      </joint>
+      <link name="${device_namespace}_infra1_frame" />
+      <joint name="${device_namespace}_infra1_to_${device_namespace}_infra1_optical_joint" type="fixed">
+        <origin xyz="0.0 0.0 0.0" rpy="${-pi/2.0} 0.0 ${-pi/2.0}" />
+        <parent link="${device_namespace}_infra1_frame" />
+        <child link="${device_namespace}_infra1_optical_frame" />
+      </joint>
+      <link name="${device_namespace}_infra1_optical_frame" />
       <!-- camera right IR joints and links -->
-      <joint name="${prefix}${name}_to_${prefix}${name}_infra2_joint" type="fixed">
+      <joint name="${device_namespace}_to_${device_namespace}_infra2_joint" type="fixed">
         <origin xyz="0.0 ${d435_cam_depth_to_infra2_offset} 0.0" rpy="0.0 0.0 0.0" />
-        <parent link="${prefix}${name}_link" />
-        <child link="${prefix}${name}_infra2_frame" />
-      </joint>
-      <link name="${prefix}${name}_infra2_frame" />
-      <joint name="${prefix}${name}_infra2_to_${prefix}${name}_infra2_optical_joint" type="fixed">
-        <origin xyz="0.0 0.0 0.0" rpy="${-pi/2.0} 0.0 ${-pi/2.0}" />
-        <parent link="${prefix}${name}_infra2_frame" />
-        <child link="${prefix}${name}_infra2_optical_frame" />
-      </joint>
-      <link name="${prefix}${name}_infra2_optical_frame" />
+        <parent link="${device_namespace}_link" />
+        <child link="${device_namespace}_infra2_frame" />
+      </joint>
+      <link name="${device_namespace}_infra2_frame" />
+      <joint name="${device_namespace}_infra2_to_${device_namespace}_infra2_optical_joint" type="fixed">
+        <origin xyz="0.0 0.0 0.0" rpy="${-pi/2.0} 0.0 ${-pi/2.0}" />
+        <parent link="${device_namespace}_infra2_frame" />
+        <child link="${device_namespace}_infra2_optical_frame" />
+      </joint>
+      <link name="${device_namespace}_infra2_optical_frame" />
       <!-- camera color joints and links -->
-      <joint name="${prefix}${name}_to_${prefix}${name}_color_joint" type="fixed">
+      <joint name="${device_namespace}_to_${device_namespace}_color_joint" type="fixed">
         <origin xyz="0.0 ${d435_cam_depth_to_color_offset} 0.0" rpy="0.0 0.0 0.0" />
-        <parent link="${prefix}${name}_link" />
-        <child link="${prefix}${name}_color_frame" />
-      </joint>
-      <link name="${prefix}${name}_color_frame" />
-      <joint name="${prefix}${name}_color_to_${prefix}${name}_color_optical_joint" type="fixed">
-        <origin xyz="0.0 0.0 0.0" rpy="${-pi/2.0} 0.0 ${-pi/2.0}" />
-        <parent link="${prefix}${name}_color_frame" />
-        <child link="${prefix}${name}_color_optical_frame" />
-      </joint>
-      <link name="${prefix}${name}_color_optical_frame" />
+        <parent link="${device_namespace}_link" />
+        <child link="${device_namespace}_color_frame" />
+      </joint>
+      <link name="${device_namespace}_color_frame" />
+      <joint name="${device_namespace}_color_to_${device_namespace}_color_optical_joint" type="fixed">
+        <origin xyz="0.0 0.0 0.0" rpy="${-pi/2.0} 0.0 ${-pi/2.0}" />
+        <parent link="${device_namespace}_color_frame" />
+        <child link="${device_namespace}_color_optical_frame" />
+      </joint>
+      <link name="${device_namespace}_color_optical_frame" />
     </xacro:if>
-    <xacro:if value="${simulation_engine == 'ignition-gazebo'}">
-      <!-- It is also possible to use single rgbd_camera sensor, but using separate rgb and depth camera
-        should be more accurate for D435 - different frames and fovs can be set -->
-      <gazebo reference="${prefix}${name}_link">
-        <!-- https://github.com/IntelRealSense/realsense-ros#published-topics -->
-        <sensor type="camera" name="${ns}{prefix}${name}_intel_realsense_d435_color">
-          <always_on>true</always_on>
-          <update_rate>30.0</update_rate>
-          <topic>${ns}${topic}/color/image_raw</topic>
-          <visualize>false</visualize>
-          <ignition_frame_id>${prefix}${name}_color_optical_frame</ignition_frame_id>
-          <horizontal_fov>${69.0/180.0*pi}</horizontal_fov>
+    <!-- It is also possible to use single rgbd_camera sensor, but using separate rgb and depth camera
+      should be more accurate for D435 - different frames and fovs can be set -->
+    <gazebo reference="${device_namespace}_link">
+      <!-- https://github.com/IntelRealSense/realsense-ros#published-topics -->
+      <sensor type="camera" name="${ns}{prefix}${device_namespace}_intel_realsense_d435_color">
+        <always_on>true</always_on>
+        <update_rate>30.0</update_rate>
+        <topic>${ns}${topic}/color/image_raw</topic>
+        <visualize>false</visualize>
+        <ignition_frame_id>${device_namespace}_color_optical_frame</ignition_frame_id>
+        <horizontal_fov>${69.0/180.0*pi}</horizontal_fov>
+        <image>
+          <width>1280</width>
+          <height>720</height>
+          <format>R8G8B8</format>
+        </image>
+        <clip>
+          <near>0.02</near>
+          <far>300.0</far>
+        </clip>
+        <ros>
+          <namespace>${ns}${device_namespace}</namespace>
+        </ros>
+      </sensor>
+      <sensor type="depth_camera" name="${ns}${device_namespace}_intel_realsense_d435_depth">
+        <always_on>true</always_on>
+        <update_rate>30.0</update_rate>
+        <topic>${ns}${topic}/depth/image_rect_raw</topic>
+        <visualize>false</visualize>
+        <ignition_frame_id>${device_namespace}_depth_optical_frame</ignition_frame_id>
+        <camera>
+          <horizontal_fov>${87.0/180.0*pi}</horizontal_fov>
           <image>
             <width>1280</width>
             <height>720</height>
-            <format>R8G8B8</format>
+            <format>R_FLOAT32</format>
           </image>
           <clip>
-            <near>0.02</near>
-            <far>300.0</far>
+            <near>0.28</near>
+            <far>8.0</far>
           </clip>
-          <ros>
-            <namespace>${ns}</namespace>
-          </ros>
-        </sensor>
-        <sensor type="depth_camera" name="${ns}${prefix}${name}_intel_realsense_d435_depth">
-          <always_on>true</always_on>
-          <update_rate>30.0</update_rate>
-          <topic>${ns}${topic}/depth/image_rect_raw</topic>
-          <visualize>false</visualize>
-          <ignition_frame_id>${prefix}${name}_depth_optical_frame</ignition_frame_id>
-          <camera>
-            <horizontal_fov>${87.0/180.0*pi}</horizontal_fov>
-            <image>
-              <width>1280</width>
-              <height>720</height>
-              <format>R_FLOAT32</format>
-            </image>
-            <clip>
-              <near>0.28</near>
-              <far>8.0</far>
-            </clip>
-            <noise>
-              <type>gaussian</type>
-              <mean>0.0</mean>
-              <stddev>0.005</stddev>
-            </noise>
-          </camera>
-          <ros>
-            <namespace>${ns}</namespace>
-          </ros>
-        </sensor>
-      </gazebo>
-    </xacro:if>
+          <noise>
+            <type>gaussian</type>
+            <mean>0.0</mean>
+            <stddev>0.005</stddev>
+          </noise>
+        </camera>
+        <ros>
+          <namespace>${ns}${device_namespace}</namespace>
+        </ros>
+      </sensor>
+    </gazebo>
   </xacro:macro>
 </robot>

File: urdf/orbbec_astra.urdf.xacro (robot description, xacro)
@@ -3,6 +3,6 @@
   <xacro:macro name="orbbec_astra"
                params="parent_link xyz rpy
-                       device_namespace:=camera
-                       namespace:=None">
+                       namespace:=None
+                       device_namespace:=camera">
     <xacro:if value="${namespace == 'None'}">
       <xacro:property name="ns" value="" />
@@ -119,5 +119,5 @@
         </camera>
         <ros>
-          <namespace>${ns}</namespace>
+          <namespace>${ns}${device_namespace}</namespace>
         </ros>
       </sensor>

File: urdf/ouster_os1_32.urdf.xacro (robot description, xacro)
@@ -91,4 +91,7 @@
         <ignition_frame_id>${ns}${prefix}os_lidar</ignition_frame_id>
         <always_on>true</always_on>
+        <ros>
+          <namespace>${ns}${device_ns}</namespace>
+        </ros>
       </sensor>
     </gazebo>

File: urdf/slamtec_rplidar_s1.urdf.xacro (robot description, xacro)
@@ -68,5 +68,5 @@
       <sensor type="gpu_lidar" name="${ns}${prefix}rplidar_s1_sensor">
         <topic>${ns}${device_ns}scan</topic>
-        <frame_id>{ns}${prefix}laser</frame_id>
+        <frame_id>${ns}${prefix}laser</frame_id>
         <ignition_frame_id>${ns}${prefix}laser</ignition_frame_id>
         <update_rate>10.0</update_rate>
