Commit message: Suggestions

File: urdf/stereolabs_zed.urdf.xacro (robot description, xacro)
@@ -21,6 +21,5 @@
     model:=zed
     namespace:=None
-    device_namespace:=None
-    ">
+    device_namespace:=zed">
     <xacro:if value="${namespace == 'None'}">
       <xacro:property name="ns" value="" />
@@ -29,10 +28,4 @@
       <xacro:property name="ns" value="${namespace}/" />
     </xacro:unless>
-    <xacro:if value="${device_namespace == 'None'}">
-      <xacro:property name="prefix" value="" />
-    </xacro:if>
-    <xacro:unless value="${device_namespace == 'None'}">
-      <xacro:property name="prefix" value="${device_namespace}_" />
-    </xacro:unless>
     <xacro:if value="${model == 'zed'}">
       <xacro:property name="baseline" value="0.12" />
@@ -84,12 +77,12 @@
     </xacro:if>
     <!-- Camera mounting point (the threaded screw hole in the bottom) -->
-    <link name="${prefix}camera_camera_link" />
-    <joint name="${prefix}camera_base_joint" type="fixed">
+    <link name="${device_namespace}_link" />
+    <joint name="${device_namespace}_base_joint" type="fixed">
       <parent link="${parent_link}" />
-      <child link="${prefix}camera_camera_link" />
+      <child link="${device_namespace}_link" />
       <origin xyz="${xyz}" rpy="${rpy}" />
     </joint>
     <!-- Camera Center -->
-    <link name="${prefix}camera_camera_center">
+    <link name="${device_namespace}_center">
       <visual>
         <origin xyz="${screw_offset_x} 0 ${screw_offset_z}" rpy="0 0 0" />
@@ -107,118 +100,116 @@
       </collision>
     </link>
-    <joint name="${prefix}camera_camera_center_joint" type="fixed">
-      <parent link="${prefix}camera_link" />
-      <child link="${prefix}camera_camera_center" />
+    <joint name="${device_namespace}_center_joint" type="fixed">
+      <parent link="${device_namespace}_link" />
+      <child link="${device_namespace}_center" />
       <origin xyz="0 0 ${height/2}" rpy="0 ${bottom_slope} 0" />
     </joint>
     <!-- Artificially Created Camera Center -->
-    <link name="${prefix}camera_center_optical_frame" />
-    <joint name="${prefix}camera_center_joint" type="fixed">
-      <parent link="${prefix}camera_camera_center" />
-      <child link="${prefix}camera_center_optical_frame" />
+    <link name="${device_namespace}_center_optical_frame" />
+    <joint name="${device_namespace}_center_joint" type="fixed">
+      <parent link="${device_namespace}_center" />
+      <child link="${device_namespace}_center_optical_frame" />
       <origin xyz="0.01 0 0" rpy="0 0 0" />
     </joint>
     <!-- Left Camera -->
-    <link name="${prefix}camera_left_camera_frame" />
-    <joint name="${prefix}camera_left_camera_joint" type="fixed">
-      <parent link="${prefix}camera_camera_center" />
-      <child link="${prefix}camera_left_camera_frame" />
+    <link name="${device_namespace}_left_camera_frame" />
+    <joint name="${device_namespace}_left_camera_joint" type="fixed">
+      <parent link="${device_namespace}_center" />
+      <child link="${device_namespace}_left_camera_frame" />
       <origin xyz="${optical_offset_x} ${baseline/2} 0" rpy="0 0 0" />
     </joint>
-    <link name="${prefix}camera_left_camera_optical_frame" />
-    <joint name="${prefix}camera_left_camera_optical_joint" type="fixed">
+    <link name="${device_namespace}_left_camera_optical_frame" />
+    <joint name="${device_namespace}_left_camera_optical_joint" type="fixed">
       <origin xyz="0 0 0" rpy="-${M_PI/2} 0.0 -${M_PI/2}" />
-      <parent link="${prefix}camera_left_camera_frame" />
-      <child link="${prefix}camera_left_camera_optical_frame" />
+      <parent link="${device_namespace}_left_camera_frame" />
+      <child link="${device_namespace}_left_camera_optical_frame" />
     </joint>
     <!-- Right Camera -->
-    <link name="${prefix}camera_right_camera_frame" />
-    <joint name="${prefix}camera_right_camera_joint" type="fixed">
-      <parent link="${prefix}camera_camera_center" />
-      <child link="${prefix}camera_right_camera_frame" />
+    <link name="${device_namespace}_right_camera_frame" />
+    <joint name="${device_namespace}_right_camera_joint" type="fixed">
+      <parent link="${device_namespace}_center" />
+      <child link="${device_namespace}_right_camera_frame" />
       <origin xyz="${optical_offset_x} -${baseline/2} 0" rpy="0 0 0" />
     </joint>
-    <link name="${prefix}camera_right_camera_optical_frame" />
-    <joint name="${prefix}camera_right_camera_optical_joint" type="fixed">
+    <link name="${device_namespace}_right_camera_optical_frame" />
+    <joint name="${device_namespace}_right_camera_optical_joint" type="fixed">
       <origin xyz="0 0 0" rpy="-${M_PI/2} 0.0 -${M_PI/2}" />
-      <parent link="${prefix}camera_right_camera_frame" />
-      <child link="${prefix}camera_right_camera_optical_frame" />
+      <parent link="${device_namespace}_right_camera_frame" />
+      <child link="${device_namespace}_right_camera_optical_frame" />
     </joint>
     <!-- ZED2 Sensors -->
     <xacro:if value="${model == 'zed2'}">
-      <link name="${prefix}camera_mag_link" />
-      <joint name="${prefix}camera_mag_joint" type="fixed">
-        <parent link="${prefix}camera_camera_center" />
-        <child link="${prefix}camera_mag_link" />
+      <link name="${device_namespace}_mag_link" />
+      <joint name="${device_namespace}_mag_joint" type="fixed">
+        <parent link="${device_namespace}_center" />
+        <child link="${device_namespace}_mag_link" />
         <origin xyz="0 0 0" rpy="0 0 0" />
       </joint>
-      <link name="${prefix}camera_baro_link" />
-      <joint name="${prefix}camera_baro_joint" type="fixed">
-        <parent link="${prefix}camera_camera_center" />
-        <child link="${prefix}camera_baro_link" />
+      <link name="${device_namespace}_baro_link" />
+      <joint name="${device_namespace}_baro_joint" type="fixed">
+        <parent link="${device_namespace}_center" />
+        <child link="${device_namespace}_baro_link" />
         <origin xyz="0 0 0" rpy="0 0 0" />
       </joint>
-      <link name="${prefix}camera_temp_left_link" />
-      <joint name="${prefix}camera_temp_left_joint" type="fixed">
-        <parent link="${prefix}camera_left_camera_frame" />
-        <child link="${prefix}camera_temp_left_link" />
+      <link name="${device_namespace}_temp_left_link" />
+      <joint name="${device_namespace}_temp_left_joint" type="fixed">
+        <parent link="${device_namespace}_left_camera_frame" />
+        <child link="${device_namespace}_temp_left_link" />
         <origin xyz="0 0 0" rpy="0 0 0" />
       </joint>
     </xacro:if>
-    <xacro:if value="${simulation_engine == 'ignition-gazebo'}">
-      <!-- It is also possible to use single rgbd_camera sensor, but using separate rgb and depth
-      camera
-        should be more accurate different frames and fovs can be set -->
-      <gazebo reference="${prefix}camera_center_optical_frame">
-        <sensor type="camera" name="${ns}${prefix}camera_stereolabs_zed_color">
-          <always_on>true</always_on>
-          <update_rate>30.0</update_rate>
-          <topic>${ns}${prefix}camera/zed_node/rgb/image_rect_color</topic>
-          <visualize>false</visualize>
-          <ignition_frame_id>${prefix}camera_center_optical_frame</ignition_frame_id>
-          <camera>
-            <horizontal_fov>${110.0/180.0*pi}</horizontal_fov>
-            <image>
-              <width>1920</width>
-              <height>1080</height>
-              <format>R8G8B8</format>
-            </image>
-            <clip>
-              <near>0.02</near>
-              <far>300.0</far>
-            </clip>
-          </camera>
-          <ros>
-            <namespace>${ns}</namespace>
-          </ros>
-        </sensor>
-        <sensor type="depth_camera" name="${ns}${prefix}camera_stereolabs_zed_depth">
-          <always_on>true</always_on>
-          <update_rate>30.0</update_rate>
-          <topic>${ns}${prefix}camera/zed_node/depth</topic>
-          <visualize>false</visualize>
-          <ignition_frame_id>${prefix}camera_center_optical_frame</ignition_frame_id>
-          <camera>
-            <horizontal_fov>${110.0/180.0*pi}</horizontal_fov>
-            <image>
-              <width>1920</width>
-              <height>1080</height>
-              <format>R_FLOAT32</format>
-            </image>
-            <clip>
-              <near>0.3</near>
-              <far>20.0</far>
-            </clip>
-            <noise type="gaussian">
-              <mean>0.0</mean>
-              <stddev>0.03</stddev>
-            </noise>
-          </camera>
-          <ros>
-            <namespace>${ns}</namespace>
-          </ros>
-        </sensor>
-      </gazebo>
-    </xacro:if>
+    <!-- It is also possible to use single rgbd_camera sensor, but using separate rgb and depth
+    camera
+      should be more accurate different frames and fovs can be set -->
+    <gazebo reference="${device_namespace}_center_optical_frame">
+      <sensor type="camera" name="${ns}${device_namespace}_stereolabs_zed_color">
+        <always_on>true</always_on>
+        <update_rate>30.0</update_rate>
+        <topic>${ns}${device_namespace}/zed_node/rgb/image_rect_color</topic>
+        <visualize>false</visualize>
+        <ignition_frame_id>${device_namespace}_center_optical_frame</ignition_frame_id>
+        <camera>
+          <horizontal_fov>${110.0/180.0*pi}</horizontal_fov>
+          <image>
+            <width>1920</width>
+            <height>1080</height>
+            <format>R8G8B8</format>
+          </image>
+          <clip>
+            <near>0.02</near>
+            <far>300.0</far>
+          </clip>
+        </camera>
+        <ros>
+          <namespace>${ns}</namespace>
+        </ros>
+      </sensor>
+      <sensor type="depth_camera" name="${ns}${device_namespace}_stereolabs_zed_depth">
+        <always_on>true</always_on>
+        <update_rate>30.0</update_rate>
+        <topic>${ns}${device_namespace}/zed_node/depth</topic>
+        <visualize>false</visualize>
+        <ignition_frame_id>${device_namespace}_center_optical_frame</ignition_frame_id>
+        <camera>
+          <horizontal_fov>${110.0/180.0*pi}</horizontal_fov>
+          <image>
+            <width>1920</width>
+            <height>1080</height>
+            <format>R_FLOAT32</format>
+          </image>
+          <clip>
+            <near>0.3</near>
+            <far>20.0</far>
+          </clip>
+          <noise type="gaussian">
+            <mean>0.0</mean>
+            <stddev>0.03</stddev>
+          </noise>
+        </camera>
+        <ros>
+          <namespace>${ns}${device_namespace}</namespace>
+        </ros>
+      </sensor>
+    </gazebo>
   </xacro:macro>
 </robot>
